Commit message: modify some function of velocity_qp from LUCAS JOSEPH auctus INRIA

File: src/franka_description_gazebo/robots/panda_arm_box.xacro (robot description, xacro)
@@ -2,5 +2,5 @@
 <robot xmlns:xacro="http://ros.org/wiki/xacro" xmlns:controller="http://playerstage.sourceforge.net/gazebo/xmlschema/#controller"   name="panda" >
   <xacro:property name="M_PI" value="3.1415926535897931" />
-  <xacro:macro name="panda_arm" params="arm_id:='panda' description_pkg:='franka_description' connected_to:='' xyz:='0 0 0' rpy:='0 0 0' gazebo_plugin:=''">
+  <xacro:macro name="panda_arm" params="arm_id:='panda' description_pkg:='franka_description_gazebo' connected_to:='' xyz:='0 0 0' rpy:='0 0 0' gazebo_plugin:=''">
     <xacro:unless value="${not connected_to}">
       <joint name="${arm_id}_joint_${connected_to}" type="fixed">
