Commit message: few changes

File: src/franka_description_gazebo/robots/hand.xacro (robot description, xacro)
@@ -12,10 +12,10 @@
       <visual>
         <geometry>
-          <mesh filename="package://franka_description/meshes/visual/hand.dae"/>
+          <mesh filename="package://franka_description_gazebo/meshes/visual/hand.dae"/>
         </geometry>
       </visual>
       <collision>
         <geometry>
-          <mesh filename="package://franka_description/meshes/collision/hand.stl"/>
+          <mesh filename="package://franka_description_gazebo/meshes/collision/hand.stl"/>
         </geometry>
       </collision>
@@ -24,10 +24,10 @@
       <visual>
         <geometry>
-          <mesh filename="package://franka_description/meshes/visual/finger.dae"/>
+          <mesh filename="package://franka_description_gazebo/meshes/visual/finger.dae"/>
         </geometry>
       </visual>
       <collision>
         <geometry>
-          <mesh filename="package://franka_description/meshes/collision/finger.stl"/>
+          <mesh filename="package://franka_description_gazebo/meshes/collision/finger.stl"/>
         </geometry>
       </collision>
@@ -37,5 +37,5 @@
         <origin xyz="0 0 0" rpy="0 0 ${pi}"/>
         <geometry>
-          <mesh filename="package://franka_description/meshes/visual/finger.dae"/>
+          <mesh filename="package://franka_description_gazebo/meshes/visual/finger.dae"/>
         </geometry>
       </visual>
@@ -43,5 +43,5 @@
         <origin xyz="0 0 0" rpy="0 0 ${pi}"/>
         <geometry>
-          <mesh filename="package://franka_description/meshes/collision/finger.stl"/>
+          <mesh filename="package://franka_description_gazebo/meshes/collision/finger.stl"/>
         </geometry>
       </collision>

File: src/franka_description_gazebo/robots/panda_arm_box.urdf.xacro (robot description, xacro)
@@ -2,6 +2,6 @@
 <robot xmlns:xacro="http://www.ros.org/wiki/xacro" name="panda">
   <xacro:arg name="gazebo_plugin" default="" />
-  <xacro:include filename="$(find franka_description)/robots/panda_arm_box.xacro" />
-  <xacro:include filename="$(find franka_description)/robots/ati.xacro" />
+  <xacro:include filename="$(find franka_description_gazebo)/robots/panda_arm_box.xacro" />
+  <xacro:include filename="$(find franka_description_gazebo)/robots/ati.xacro" />
   <xacro:panda_arm gazebo_plugin="$(arg gazebo_plugin)"/>
 <!--   <xacro:ati /> -->

File: src/franka_description_gazebo/robots/panda_arm_hand.urdf.xacro (robot description, xacro)
@@ -2,6 +2,6 @@
 <robot xmlns:xacro="http://www.ros.org/wiki/xacro" name="panda">
   <xacro:arg name="gazebo_plugin" default="" />
-  <xacro:include filename="$(find franka_description)/robots/panda_arm.xacro"/>
-  <xacro:include filename="$(find franka_description)/robots/hand.xacro"/>
+  <xacro:include filename="$(find franka_description_gazebo)/robots/panda_arm.xacro"/>
+  <xacro:include filename="$(find franka_description_gazebo)/robots/hand.xacro"/>
   <xacro:panda_arm gazebo_plugin="$(arg gazebo_plugin)"/>
   <xacro:hand ns="panda" rpy="0 0 ${-pi/4}" connected_to="panda_link8"/>
